Commit message: update files

File: urdf/gz_control.xacro (robot description, xacro)
@@ -3,5 +3,5 @@
   <gazebo>
     <plugin filename="gz-sim-diff-drive-system" name="gz::sim::systems::DiffDrive">
-      <left_joint>drivewhl_l_joint</left_joint>
+      <!-- <left_joint>drivewhl_l_joint</left_joint>
       <right_joint>drivewhl_r_joint</right_joint>
       <wheel_separation>0.4</wheel_separation>
@@ -9,6 +9,31 @@
       <odom_frame>odom</odom_frame>
       <robot_base_frame>base_link</robot_base_frame>
+      <publish_tf>true</publish_tf>
+      <tf_topic>/tf</tf_topic>
+      <tf_topic>/tf</tf_topic>
+      <frame_id>odom</frame_id>
+      <child_frame_id>base_link</child_frame_id>
       <topic>/cmd_vel</topic>
+      <odom_topic>/odom</odom_topic> -->
+            <!-- Wheel joints -->
+      <left_joint>drivewhl_l_joint</left_joint>
+      <right_joint>drivewhl_r_joint</right_joint>
+      <!-- Geometry -->
+      <wheel_separation>0.40</wheel_separation>
+      <wheel_radius>0.10</wheel_radius>
+      <!-- Odometry -->
+      <odom_publish_frequency>50</odom_publish_frequency>
       <odom_topic>/odom</odom_topic>
+      <!-- TF publishing -->
+      <tf_topic>/tf</tf_topic>
+      <frame_id>odom</frame_id>
+      <child_frame_id>base_link</child_frame_id>
+      <!-- Command velocity -->
+      <topic>/cmd_vel</topic>
+      <!-- Optional limits (safe defaults) -->
+      <max_linear_velocity>1.0</max_linear_velocity>
+      <max_angular_velocity>2.0</max_angular_velocity>
+      <max_linear_acceleration>2.0</max_linear_acceleration>
+      <max_angular_acceleration>4.0</max_angular_acceleration>
     </plugin>
   </gazebo>

File: urdf/gz_sensors.xacro (robot description, xacro)
@@ -9,4 +9,6 @@
       name="gz::sim::systems::Imu">
     </plugin>
+    <!-- <plugin filename="gz-sim-lidar-system"
+        name="gz::sim::systems::Lidar"/> -->
     <!-- ===================== JOINT STATE PUBLISHER ===================== -->
     <plugin filename="gz-sim-joint-state-publisher-system"
@@ -92,6 +94,6 @@
             <samples>360</samples>
             <resolution>1.00000</resolution>
-            <min_angle>-3.14</min_angle>
-            <max_angle>3.14</max_angle>
+            <min_angle>0.00000</min_angle>
+            <max_angle>6.280000</max_angle>
           </horizontal>
         </scan>
@@ -113,16 +115,18 @@
     <sensor name="depth_camera" type="depth_camera">
       <!-- <topic>/camera/image</topic> -->
-      <topic>camera</topic>
-      <camera_info_topic>/camera/camera_info</camera_info_topic>
+      <!-- <topic>depth_camera</topic> -->
+      <topic>/camera/depth/image_raw</topic>
+      <!-- <camera_info_topic>/camera/camera_info</camera_info_topic> -->
       <always_on>true</always_on>
       <update_rate>30</update_rate>
       <visualize>true</visualize>
-      <ignition_frame_id>camera_depth_frame</ignition_frame_id>
+      <!-- <ignition_frame_id>camera_depth_frame</ignition_frame_id> -->
       <camera>
-        <horizontal_fov>1.0</horizontal_fov>
+        <frame_id>camera_depth_frame</frame_id>
+        <horizontal_fov>1.047198</horizontal_fov>
         <image>
           <width>640</width>
           <height>480</height>
-          <format>R8G8B8</format>
+          <format>R_FLOAT32</format>
         </image>
         <clip>

File: urdf/robot_gz.urdf.xacro (robot description, xacro)
@@ -10,4 +10,5 @@
   <!-- Plugins de sensores para GZ -->
   <xacro:include filename="gz_sensors.xacro"/>
+  <xacro:include filename="gz_physics.xacro"/>
   <!-- Control diferencial: GZ puro o ros2_control -->
   <xacro:if value="$(arg use_ros2_control)">

File: urdf/sensors.xacro (robot description, xacro)
@@ -88,5 +88,6 @@
     <parent link="camera_link"/>
     <child link="camera_depth_frame"/>
-    <origin xyz="0 0 0" rpy="${-pi/2} 0 ${-pi/2}"/>
+    <!-- <origin xyz="0.02 0 0" rpy="${-pi/2} 0 ${-pi/2}"/> -->
+    <origin xyz="0.002 0 0" rpy="0 0 0"/>
   </joint>
 </xacro:robot>
